File: comms_board/comms_board.kicad_sch (KiCad schematic)
At the start: 46 parts, among them J1 X6, J10 USB to UART Conn, J2 X4, J3 X5, J4 X7, J5 X9 LOCAL CAN Feedthrough Conn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, J6 X8: LOCAL CAN Host Interface, J7 Pins to select 120 terminal r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, J8 UPDI Friend Input Terminal, Q1 MMBT3904, Q2 MMBT3906, Q3 2N7002, Q4 Q_Dual_NPN_NPN_E1B1C2E2B2C1, SW1 DIP Switch, U10 REF3040 4.096 Ref Voltage, U13 AVR128DB48x-xPT, U2 LTV-817S, U3 INA826, U4 MCP25625 - CAN Transciever, U5 L7812 +12V Lin Reg, U6 L7912 -12V Lin Reg, U7 L7805 +5V Lin Reg, U8 OPA2140, U9 LM358, Y1 16MHz CXO

Commit message: so much! I should push more!
Parts:
- removed C10, C9: 27pF, Capacitor_SMD:C_1206_3216Metric_Pad1.33x1.80mm_HandSolder, symbol Device:C
- removed C13, C14, C15, C16, C17, C18: 100n, Capacitor_SMD:C_1206_3216Metric_Pad1.33x1.80mm_HandSolder, symbol Device:C
- removed FL1: Common Mode Choke, Inductor_SMD:L_CommonMode_Wurth_WE-CNSW-1206, symbol Filter:Choke_CommonMode_FerriteCore_1243
- removed J10: USB to UART Conn, symbol Connector:Conn_01x06_Pin
- removed J5: X9 LOCAL CAN Feedthrough Connector, Connector_Dsub:DSUB-9_Pins_Horizontal_P2.77x2.84mm_EdgePinOffset9.40mm, symbol Connector:DE9_Pins
- removed J6: X8: LOCAL CAN Host Interface, Connector_Dsub:DSUB-9_Pins_Horizontal_P2.77x2.84mm_EdgePinOffset9.40mm, symbol Connector:DE9_Pins
- removed J7: Pins to select 120 terminal resistance or not, TerminalBlock:TerminalBlock_MaiXu_MX126-5.0-03P_1x03_P5.00mm, symbol Connector:Conn_01x03_Pin
- removed J8: UPDI Friend Input Terminal, symbol Connector:Screw_Terminal_01x03
- removed R3: 120, symbol Device:R_US
- removed SW1: DIP Switch, Button_Switch_THT:Nidec_Copal_SH-7010C, symbol Switch:SW_Coded_SH-7030
- removed U13: AVR128DB48x-xPT, Package_QFP:TQFP-48_7x7mm_P0.5mm, symbol MCU_Microchip_AVR_Dx:AVR128DB48x-xPT
- removed U4: MCP25625 - CAN Transciever, Package_SO:SSOP-28_5.3x10.2mm_P0.65mm, symbol Interface_CAN_LIN:MCP25625x-x-SS
- removed Y1: 16MHz CXO, Crystal:Crystal_SMD_3225-4Pin_3.2x2.5mm, symbol Oscillator:SG-210SCD
- added C19, C20, C21, C24, C25, C26: 100n, Capacitor_SMD:C_0805_2012Metric_Pad1.18x1.45mm_HandSolder, symbol Device:C
- added C22, C23: 27p, Capacitor_SMD:C_1206_3216Metric_Pad1.33x1.80mm_HandSolder, symbol Device:C
- added D6: Red LED, LED_THT:LED_D1.8mm_W3.3mm_H2.4mm, symbol Device:LED
- added D7: Yellow LED, LED_THT:LED_D1.8mm_W3.3mm_H2.4mm, symbol Device:LED
- added D8: Green LED, LED_THT:LED_D1.8mm_W3.3mm_H2.4mm, symbol Device:LED
- added FL2: Common Mode Choke, Inductor_SMD:L_CommonMode_Wurth_WE-CNSW-1206, symbol Filter:Choke_CommonMode_FerriteCore_1243
- added J11: X8: LOCAL CAN Host Interface, dsub:CONN_DE09-SL-24_ADM_DSUB, symbol dsub_with_mounts:DE9_Pins
- added J12: Pins to select 120 terminal resistance or not, Connector_PinHeader_2.54mm:PinHeader_1x03_P2.54mm_Vertical, symbol Connector:Conn_01x03_Pin
- added J13: CXO TP, Connector_PinHeader_2.54mm:PinHeader_1x01_P2.54mm_Vertical, symbol Connector:Conn_01x01_Pin
- added J14: CXO TP GND, Connector_PinHeader_2.54mm:PinHeader_1x01_P2.54mm_Vertical, symbol Connector:Conn_01x01_Pin
- added J15: Conn_01x02_Pin, TerminalBlock:TerminalBlock_MaiXu_MX126-5.0-02P_1x02_P5.00mm, symbol Connector:Conn_01x02_Pin
- added J16: UPDI Friend Input Terminal, TerminalBlock:TerminalBlock_MaiXu_MX126-5.0-03P_1x03_P5.00mm, symbol Connector:Screw_Terminal_01x03
- added J17: USB to UART Conn, Connector_PinHeader_2.54mm:PinHeader_1x06_P2.54mm_Vertical, symbol Connector:Conn_01x06_Pin
- added J9: X8: LOCAL CAN Host Interface, dsub:CONN_DE09-SL-24_ADM_DSUB, symbol Connector:DE9_Pins
- added R4: 120, Resistor_SMD:R_1206_3216Metric_Pad1.30x1.75mm_HandSolder, symbol Device:R_US
- added R5, R6, R7: 330, Resistor_SMD:R_1206_3216Metric_Pad1.30x1.75mm_HandSolder, symbol Device:R_US
- added SW2: DIP Switch, Button_Switch_THT:Nidec_Copal_SH-7010C, symbol Switch:SW_Coded_SH-7030
- added U14: MCP25625 - CAN Transciever, Package_SO:SSOP-28_5.3x10.2mm_P0.65mm, symbol Interface_CAN_LIN:MCP25625x-x-SS
- added U15: AVR128DB48x-xPT, Package_QFP:TQFP-48_7x7mm_P0.5mm, symbol MCU_Microchip_AVR_Dx:AVR128DB48x-xPT
- added Y2: Crystal_GND24, Crystal:Crystal_SMD_3225-4Pin_3.2x2.5mm, symbol Device:Crystal_GND24
Connections:
- net +5V: now also C19.1, C20.1, C21.1, C24.2, C25.1, C26.2, J15.1 (Pin_1), U14.1 (V_{IO}), U14.19 (V_{DD}), U14.27 (V_{DDA}), U15.14 (VDDIO2), U15.28 (AVDD), U15.42 (VDD)
- net CAN H: now also FL2.1, J11.7, J9.7
- net CAN H FILT: now also FL2.2, R4.2, U14.4 (CANH)
- net CAN L: now also FL2.4, J11.2, J9.2
- net CAN L FILT: now also FL2.3, J12.1 (Pin_1), U14.3 (CANL)
- net CS: now also U14.17 (~{CS}), U15.47 (PA3)
- net GND: now also C19.2, C20.2, C21.2, C22.1, C23.1, C24.1, C25.2, C26.1, D6.1 (K), D7.1 (K), D8.1 (K), J11.10, J11.11, J11.3, J11.6, J14.1 (Pin_1), J15.2 (Pin_2), J16.1 (Pin_1), J17.1 (Pin_1), J9.10, J9.11, J9.3, J9.6, SW2.C, U14.10 (GND), U14.5 (STBY), U15.15 (GND), U15.29 (AGND), U15.43 (GND), Y2.2 (G), Y2.4 (G)
- net INT: now also U14.13 (~{INT}), U15.4 (PB0)
- net MISO: now also U14.16 (SO), U15.1 (PA5)
- net MOSI: now also U14.15 (SI), U15.48 (PA4)
- net RESET: now also U14.18 (~{RESET})
- net RX: now also J17.5 (Pin_5), U15.44 (XTALHF1/PA0)
- net SCK: now also U14.14 (SCK), U15.2 (PA6)
- net TX: now also J17.4 (Pin_4), U15.45 (XTALHF2/PA1)
- net UPDI Wire: now also J16.3 (Pin_3), U15.41 (UPDI)
- new net: SW2.1, U15.23 (PD3)
- new net: SW2.2, U15.21 (PD1)
- new net: SW2.4, U15.22 (PD2)
- new net: SW2.8, U15.24 (PD4)
- new net: D6.2 (A), R5.2
- new net: C22.2, U14.9 (OSC1), Y2.1
- new net: D7.2 (A), R6.2
- new net: R5.1, U15.10 (PC0)
- new net: R6.1, U15.11 (PC1)
- new net: R7.1, U15.12 (PC2)
- new net: C23.2, U14.8 (OSC2), Y2.3
- new net: U14.20 (TxCAN), U14.24 (T_{XD})
- new net: U14.21 (RxCAN), U14.28 (R_{XD})
- new net: J13.1 (Pin_1), U14.22 (CLKOUT)
- new net: J12.2 (Pin_2), J12.3 (Pin_3), R4.1
- new net: D8.2 (A), R7.2
- no-connect marks 4 -> 37
Other:
- note added: "Wiring to signify ID to scream into CAN. Pull down. truth table in datasheet. Wiring wonky to make the PCB layout smoother"
- note removed: "Wiring to signify ID to scream into CAN. Pull down. truth table in datasheet"
- moved on the sheet: C11, C12, U10, U7
