File: can_tester/can_tester.kicad_pcb (KiCad board)
At the start: 2 copper layers, 100 x 73 mm, 20 parts, among them J1 Conn_01x02_Pin, J10 USB to UART Conn, J5 X9 LOCAL CAN Feedthrough Conn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, J6 X8: LOCAL CAN Host Interface, J7 Pins to select 120 terminal r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, J8 UPDI Friend Input Terminal, SW1 DIP Switch, U13 AVR128DB48x-xPT, U4 MCP25625 - CAN Transciever, Y2 Crystal_GND24

Commit message: can tester board complete?:
Parts:
- added C10: 27p, Capacitor_SMD:C_0603_1608Metric_Pad1.08x0.95mm_HandSolder, F.Cu at (94.3, 34.2)
- added C13: 100n, Capacitor_SMD:C_0603_1608Metric_Pad1.08x0.95mm_HandSolder, F.Cu at (79.2, 33.1)
- added C14: 100n, Capacitor_SMD:C_0603_1608Metric_Pad1.08x0.95mm_HandSolder, F.Cu at (91.2, 42.5)
- added C15: 100n, Capacitor_SMD:C_0603_1608Metric_Pad1.08x0.95mm_HandSolder, F.Cu at (79.1, 38.6)
- added C16: 100n, Capacitor_SMD:C_0603_1608Metric_Pad1.08x0.95mm_HandSolder, F.Cu at (115.9, 35.7)
- added C17: 100n, Capacitor_SMD:C_0603_1608Metric_Pad1.08x0.95mm_HandSolder, F.Cu at (110.2, 26.2)
- added C18: 100n, Capacitor_SMD:C_0603_1608Metric_Pad1.08x0.95mm_HandSolder, F.Cu at (106.7, 41.1)
- added C9: 27p, Capacitor_SMD:C_0603_1608Metric_Pad1.08x0.95mm_HandSolder, F.Cu at (101.2, 34.2)
- added D1: Red LED, LED_THT:LED_D1.8mm_W3.3mm_H2.4mm, F.Cu at (107.7, 58.4)
- added D1: Red LED, LED_THT:LED_D1.8mm_W3.3mm_H2.4mm, F.Cu at (107.5, 145.8)
- added D2: Yellow LED, LED_THT:LED_D1.8mm_W3.3mm_H2.4mm, F.Cu at (111.8, 58.4)
- added D2: Yellow LED, LED_THT:LED_D1.8mm_W3.3mm_H2.4mm, F.Cu at (111.6, 145.8)
- added D3: Green LED, LED_THT:LED_D1.8mm_W3.3mm_H2.4mm, F.Cu at (115.7, 145.8)
- added D3: Green LED, LED_THT:LED_D1.8mm_W3.3mm_H2.4mm, F.Cu at (115.9, 58.4)
- added FL1: Common Mode Choke, Inductor_SMD:L_CommonMode_Wurth_WE-CNSW-1206, F.Cu at (79.2, 47.6)
- added J1: Conn_01x02_Pin, TerminalBlock:TerminalBlock_MaiXu_MX126-5.0-02P_1x02_P5.00mm, F.Cu at (88.5, 6.07)
- added J10: USB to UART Conn, TerminalBlock:TerminalBlock_MaiXu_MX126-5.0-06P_1x06_P5.00mm, F.Cu at (136.4, 19.1)
- added J3: CXO TP, Connector_PinHeader_2.54mm:PinHeader_1x01_P2.54mm_Vertical, F.Cu at (81.2, 35.8)
- added J3: CXO TP, Connector_PinHeader_2.54mm:PinHeader_1x01_P2.54mm_Vertical, F.Cu at (81.0, 123.2)
- added J5: X9 LOCAL CAN Feedthrough Connector, Connector_Dsub:DSUB-9_Pins_Horizontal_P2.77x2.84mm_EdgePinOffset9.40mm, B.Cu at (67.9, 45.6)
- added J6: X8: LOCAL CAN Host Interface, Connector_Dsub:DSUB-9_Pins_Horizontal_P2.77x2.84mm_EdgePinOffset9.40mm, B.Cu at (67.9, 13.1)
- added J7: Pins to select 120 terminal resistance or not, TerminalBlock:TerminalBlock_MaiXu_MX126-5.0-03P_1x03_P5.00mm, F.Cu at (85.7, 55.1)
- added J8: UPDI Friend Input Terminal, TerminalBlock:TerminalBlock_MaiXu_MX126-5.0-03P_1x03_P5.00mm, F.Cu at (135.4, 39.2)
- added R3: 120, Resistor_SMD:R_1206_3216Metric_Pad1.30x1.75mm_HandSolder, F.Cu at (101.2, 54.5)
- added R4: 330, Resistor_SMD:R_1206_3216Metric_Pad1.30x1.75mm_HandSolder, F.Cu at (107.4, 51.2)
- added R4: 330, Resistor_SMD:R_1206_3216Metric_Pad1.30x1.75mm_HandSolder, F.Cu at (107.2, 138.6)
- added R5: 330, Resistor_SMD:R_1206_3216Metric_Pad1.30x1.75mm_HandSolder, F.Cu at (110.7, 51.2)
- added R5: 330, Resistor_SMD:R_1206_3216Metric_Pad1.30x1.75mm_HandSolder, F.Cu at (110.5, 138.6)
- added R6: 330, Resistor_SMD:R_1206_3216Metric_Pad1.30x1.75mm_HandSolder, F.Cu at (114.0, 51.2)
- added R6: 330, Resistor_SMD:R_1206_3216Metric_Pad1.30x1.75mm_HandSolder, F.Cu at (113.8, 138.6)
- added REF**: MountingHole_2.7mm, MountingHole:MountingHole_2.7mm, F.Cu at (60.4, 145.0)
- added REF**: MountingHole_2.7mm, MountingHole:MountingHole_2.7mm, F.Cu at (150.2, -6.20)
- added REF**: MountingHole_2.7mm, MountingHole:MountingHole_2.7mm, F.Cu at (150.0, 81.2)
- added REF**: MountingHole_2.7mm, MountingHole:MountingHole_2.7mm, F.Cu at (60.6, -6.20)
- added REF**: MountingHole_2.7mm, MountingHole:MountingHole_2.7mm, F.Cu at (60.6, 57.6)
- added REF**: MountingHole_2.7mm, MountingHole:MountingHole_2.7mm, F.Cu at (150.0, 145.2)
- added REF**: MountingHole_2.7mm, MountingHole:MountingHole_2.7mm, F.Cu at (150.2, 57.8)
- added REF**: MountingHole_2.7mm, MountingHole:MountingHole_2.7mm, F.Cu at (60.4, 81.2)
- added SW1: DIP Switch, Button_Switch_THT:Nidec_Copal_SH-7010C, F.Cu at (117.9, 39.7)
- added U13: AVR128DB48x-xPT, Package_QFP:TQFP-48_7x7mm_P0.5mm, F.Cu at (109.2, 33.6)
- added U4: MCP25625 - CAN Transciever, Package_SO:SSOP-28_5.3x10.2mm_P0.65mm, F.Cu at (87.7, 34.8)
- added Y2: Crystal_GND24, Crystal:Crystal_SMD_3225-4Pin_3.2x2.5mm, F.Cu at (97.8, 34.5)
- J5, J6: moved to B.Cu
- moved J6 11.1 mm to (67.7, 100.5), turned to 90 degrees
- moved J5 11.1 mm to (67.7, 133.0), turned to 90 degrees
Connections:
- U13 pad 10: unconnected-(U13-PC0-Pad10) -> Net-(U13-PC0)
- U13 pad 11: unconnected-(U13-PC1-Pad11) -> Net-(U13-PC1)
- U13 pad 12: unconnected-(U13-PC2-Pad12) -> Net-(U13-PC2)
- U4 pad 22: unconnected-(U4-CLKOUT-Pad22) -> Net-(J3-Pin_1)
Routing:
- net +5V: track 214.2 -> 428.1 mm
- net GND: track 65.3 -> 156.8 mm
- net /CAN H: track 50.2 -> 111.7 mm
- net /CAN L: track 50.2 -> 91.1 mm
- net /CAN H FILT: track 37.5 -> 75.0 mm
- net Net-(U13-PC2): track 0.00 -> 35.3 mm
- net Net-(U13-PC1): track 0.00 -> 35.2 mm
- net Net-(U13-PC0): track 0.00 -> 34.6 mm
- net /CAN L FILT: track 34.6 -> 69.1 mm
- net /CS: track 28.5 -> 57.0 mm
- net /UPDI Wire: track 26.8 -> 53.6 mm
- net /TX: track 24.6 -> 49.2 mm
- net /MOSI: track 23.0 -> 45.9 mm
- net /MISO: track 22.0 -> 44.0 mm
- net Net-(U13-PD1): track 20.1 -> 40.2 mm
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Other:
- board size 100 x 73 mm -> 100.2 x 160.4 mm
- board text added: "5V GND"
- board text added: "UPDI X GND"
- board text added: "X RX TX X X GND"
- board text added: "X8"
- board text added: "X9"
