File: can_tester/can_tester.kicad_pcb (KiCad board)
At the start: 2 copper layers, 100.2 x 160.4 mm, 62 parts, among them J1 Conn_01x02_Pin, J10 USB to UART Conn, J3 CXO TP, J5 X9 LOCAL CAN Feedthrough Conn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, J6 X8: LOCAL CAN Host Interface, J7 Pins to select 120 terminal r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, J8 UPDI Friend Input Terminal, SW1 DIP Switch, U13 AVR128DB48x-xPT, U4 MCP25625 - CAN Transciever, Y2 Crystal_GND24

Commit message: so much! I should push more!
Parts:
- removed the C10 at (94.3, 34.2)
- removed the C13 at (79.2, 33.1)
- removed the C14 at (91.2, 42.5)
- removed the C15 at (79.1, 38.6)
- removed the C16 at (115.9, 35.7)
- removed the C17 at (110.2, 26.2)
- removed the C18 at (106.7, 41.1)
- removed the C9 at (101.2, 34.2)
- removed the D1 at (107.7, 58.4)
- removed the D2 at (111.8, 58.4)
- removed the D3 at (115.9, 58.4)
- removed the FL1 at (79.2, 47.6)
- removed the J1 at (88.5, 6.07)
- removed the J10 at (136.4, 19.1)
- removed the J3 at (81.2, 35.8)
- removed J5 (x2): X9 LOCAL CAN Feedthrough Connector, Connector_Dsub:DSUB-9_Pins_Horizontal_P2.77x2.84mm_EdgePinOffset9.40mm
- removed the J6 at (67.9, 13.1)
- removed the J7 at (85.7, 55.1)
- removed the J8 at (135.4, 39.2)
- removed the R3 at (101.2, 54.5)
- removed the R4 at (107.4, 51.2)
- removed the R5 at (110.7, 51.2)
- removed the R6 at (114.0, 51.2)
- removed the REF** at (150.2, -6.20)
- removed the REF** at (60.6, -6.20)
- removed the REF** at (60.6, 57.6)
- removed the REF** at (150.2, 57.8)
- removed the SW1 at (117.9, 39.7)
- removed the U13 at (109.2, 33.6)
- removed the U4 at (87.7, 34.8)
- removed the U4 at (87.5, 122.2)
- removed the Y2 at (97.8, 34.5)
- added J13: CANL TP, Connector_PinHeader_2.54mm:PinHeader_1x02_P2.54mm_Vertical, F.Cu at (72.6, 121.9)
- added J14: CANH TP, Connector_PinHeader_2.54mm:PinHeader_1x02_P2.54mm_Vertical, F.Cu at (69.4, 128.4)
- added J15: FILT CANL TP, Connector_PinHeader_2.54mm:PinHeader_1x02_P2.54mm_Vertical, F.Cu at (81.6, 142.5)
- added J16: FILT CANH TP, Connector_PinHeader_2.54mm:PinHeader_1x02_P2.54mm_Vertical, F.Cu at (86.9, 136.6)
- added J17: GND Conn, Connector_PinHeader_2.54mm:PinHeader_1x02_P2.54mm_Vertical, F.Cu at (106.6, 124.0)
- added J18: GND Conn, Connector_PinHeader_2.54mm:PinHeader_1x02_P2.54mm_Vertical, F.Cu at (86.9, 108.6)
- added J2: X9: LOCAL CAN Host Interface, dsub:CONN_DE09-SL-24_ADM_DSUB, F.Cu at (55.8, 110.2)
- added U4: MCP25625 - CAN Transciever, Package_SO:SSOP-28_5.3x10.2mm_P0.65mm, F.Cu at (87.5, 122.2)
- C10, C9: footprint Capacitor_SMD:C_0603_1608Metric_Pad1.08x0.95mm_HandSolder -> Capacitor_SMD:C_1206_3216Metric_Pad1.33x1.80mm_HandSolder
- C13, C14, C15, C16, C17, C18: footprint Capacitor_SMD:C_0603_1608Metric_Pad1.08x0.95mm_HandSolder -> Capacitor_SMD:C_0805_2012Metric_Pad1.18x1.45mm_HandSolder
- J10: footprint TerminalBlock:TerminalBlock_MaiXu_MX126-5.0-06P_1x06_P5.00mm -> Connector_PinHeader_2.54mm:PinHeader_1x06_P2.54mm_Vertical
- J6: footprint Connector_Dsub:DSUB-9_Pins_Horizontal_P2.77x2.84mm_EdgePinOffset9.40mm -> dsub:CONN_DE09-SL-24_ADM_DSUB; moved to F.Cu
- J7: footprint TerminalBlock:TerminalBlock_MaiXu_MX126-5.0-03P_1x03_P5.00mm -> Connector_PinHeader_2.54mm:PinHeader_1x03_P2.54mm_Vertical
- R3: footprint Resistor_SMD:R_1206_3216Metric_Pad1.30x1.75mm_HandSolder -> Resistor_THT:R_Axial_DIN0204_L3.6mm_D1.6mm_P2.54mm_Vertical
- SW1: moved to B.Cu
- moved J6 27.5 mm to (85.2, 79.3), turned to 0 degrees
- moved SW1 19.9 mm to (136.5, 133.7), turned to 180 degrees
- moved C16 17.7 mm to (133.4, 123.4)
- moved C17 17.6 mm to (127.6, 114.0), turned to 180 degrees
- moved C18 17.5 mm to (124.0, 129.0)
- moved U13 17.3 mm to (126.2, 121.0)
- moved J8 9.19 mm to (144.4, 127.0)
- moved J1 8.73 mm to (88.2, 102.2)
- moved R3 7.25 mm to (93.8, 142.8)
- moved D1 7.02 mm to (113.1, 141.6)
- moved D3 7.02 mm to (121.3, 141.6)
- moved R6 7.02 mm to (119.4, 134.4)
- moved D2 7.02 mm to (117.2, 141.6)
- moved R4 7.02 mm to (112.8, 134.4)
- moved R5 7.02 mm to (116.1, 134.4)
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Connections:
- SW1 pad 1: Net-(U13-PD3) -> Net-(U13-PD4)
- SW1 pad 4: Net-(U13-PD2) -> Net-(U13-PD3)
- SW1 pad 8: Net-(U13-PD4) -> Net-(U13-PD2)
- U13 pad 46: unconnected-(U13-PA2-Pad46) -> /RESET
- U13 pad 6: unconnected-(U13-PB2-Pad6) -> /Rx0
- U13 pad 7: unconnected-(U13-PB3-Pad7) -> /Rx1
- U13 pad 8: unconnected-(U13-PB4-Pad8) -> /STBY
Routing:
- net +5V: track 428.1 -> 227.3 mm
- net /RESET: track 0.00 -> 49.2 mm
- net /CAN H: track 111.7 -> 72.4 mm
- net /CAN H FILT: track 75.0 -> 37.3 mm
- net /UPDI Wire: track 53.6 -> 18.7 mm
- net /TX: track 49.2 -> 15.1 mm
- net /Rx1: track 0.00 -> 33.1 mm
- net /STBY: track 0.00 -> 33.1 mm
- net /Rx0: track 0.00 -> 33.0 mm
- net /CAN L FILT: track 69.1 -> 41.2 mm
- net /CAN L: track 91.1 -> 65.0 mm
- net Net-(U13-PD1): track 40.2 -> 14.3 mm
- net Net-(U13-PC2): track 35.3 -> 10.3 mm
- net Net-(U13-PC1): track 35.2 -> 13.1 mm
- net Net-(U13-PC0): track 34.6 -> 15.0 mm
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Other:
- board size 100.2 x 160.4 mm -> 100 x 71 mm
- board text added: "x RX TX x x GND"
- board text removed: "X RX TX X X GND"
