File: can_tester/can_tester.kicad_sch (KiCad schematic)
At the start: 0 parts

Commit message: finished comms test board?
Parts:
- added C10, C9: 27p, Capacitor_SMD:C_0603_1608Metric_Pad1.08x0.95mm_HandSolder, symbol Device:C
- added C13, C14, C15, C16, C17, C18: 100n, Capacitor_SMD:C_0603_1608Metric_Pad1.08x0.95mm_HandSolder, symbol Device:C
- added FL1: Common Mode Choke, Inductor_SMD:L_CommonMode_Wurth_WE-CNSW-1206, symbol Filter:Choke_CommonMode_FerriteCore_1243
- added J1: Conn_01x02_Pin, TerminalBlock:TerminalBlock_MaiXu_MX126-5.0-02P_1x02_P5.00mm, symbol Connector:Conn_01x02_Pin
- added J10: USB to UART Conn, TerminalBlock:TerminalBlock_MaiXu_MX126-5.0-06P_1x06_P5.00mm, symbol Connector:Conn_01x06_Pin
- added J5: X9 LOCAL CAN Feedthrough Connector, Connector_Dsub:DSUB-9_Pins_Horizontal_P2.77x2.84mm_EdgePinOffset9.40mm, symbol Connector:DE9_Pins
- added J6: X8: LOCAL CAN Host Interface, Connector_Dsub:DSUB-9_Pins_Horizontal_P2.77x2.84mm_EdgePinOffset9.40mm, symbol Connector:DE9_Pins
- added J7: Pins to select 120 terminal resistance or not, TerminalBlock:TerminalBlock_MaiXu_MX126-5.0-03P_1x03_P5.00mm, symbol Connector:Conn_01x03_Pin
- added J8: UPDI Friend Input Terminal, TerminalBlock:TerminalBlock_MaiXu_MX126-5.0-03P_1x03_P5.00mm, symbol Connector:Screw_Terminal_01x03
- added R3: 120, Resistor_SMD:R_1206_3216Metric_Pad1.30x1.75mm_HandSolder, symbol Device:R_US
- added SW1: DIP Switch, Button_Switch_THT:Nidec_Copal_SH-7010C, symbol Switch:SW_Coded_SH-7030
- added U13: AVR128DB48x-xPT, Package_QFP:TQFP-48_7x7mm_P0.5mm, symbol MCU_Microchip_AVR_Dx:AVR128DB48x-xPT
- added U4: MCP25625 - CAN Transciever, Package_SO:SSOP-28_5.3x10.2mm_P0.65mm, symbol Interface_CAN_LIN:MCP25625x-x-SS
- added Y2: Crystal_GND24, Crystal:Crystal_SMD_3225-4Pin_3.2x2.5mm, symbol Device:Crystal_GND24
Connections:
- new net: C9.2, U4.9 (OSC1), Y2.1
- new net: C10.2, U4.8 (OSC2), Y2.3
- new net: SW1.2, U13.21 (PD1)
- new net: SW1.4, U13.22 (PD2)
- new net: SW1.1, U13.23 (PD3)
- new net: SW1.8, U13.24 (PD4)
- new net: U4.20 (TxCAN), U4.24 (T_{XD})
- new net: U4.21 (RxCAN), U4.28 (R_{XD})
- new net: J7.2 (Pin_2), J7.3 (Pin_3), R3.1
- new net +5V: C13.1, C14.1, C15.1, C16.2, C17.2, C18.1, J1.1 (Pin_1), U13.14 (VDDIO2), U13.28 (AVDD), U13.42 (VDD), U4.1 (V_{IO}), U4.19 (V_{DD}), U4.27 (V_{DDA})
- new net CAN H: FL1.1, J5.7, J6.7
- new net CAN H FILT: FL1.2, R3.2, U4.4 (CANH)
- new net CAN L: FL1.4, J5.2, J6.2
- new net CAN L FILT: FL1.3, J7.1 (Pin_1), U4.3 (CANL)
- new net CS: U13.47 (PA3), U4.17 (~{CS})
- new net GND: C10.1, C13.2, C14.2, C15.2, C16.1, C17.1, C18.2, C9.1, J1.2 (Pin_2), J10.1 (Pin_1), J5.3, J5.6, J6.3, J6.6, J8.1 (Pin_1), SW1.C, U13.15 (GND), U13.29 (AGND), U13.43 (GND), U4.10 (GND), U4.5 (STBY), Y2.2 (G), Y2.4 (G)
- new net INT: U13.4 (PB0), U4.13 (~{INT})
- new net MISO: U13.1 (PA5), U4.16 (SO)
- new net MOSI: U13.48 (PA4), U4.15 (SI)
- new net RESET: U4.18 (~{RESET})
- new net RX: J10.5 (Pin_5), U13.44 (XTALHF1/PA0)
- new net SCK: U13.2 (PA6), U4.14 (SCK)
- new net TX: J10.4 (Pin_4), U13.45 (XTALHF2/PA1)
- new net UPDI Wire: J8.3 (Pin_3), U13.41 (UPDI)
- no-connect marks 0 -> 41
Other:
- note added: "This breakout board will be for writing code to AVR"
- note added: "Wiring to signify ID to scream into CAN. Pull down. truth table in datasheet. Wiring wonky to make the PCB layout smoother"

Commit message: can tester board complete?:
Parts:
- added D1: Red LED, LED_THT:LED_D1.8mm_W3.3mm_H2.4mm, symbol Device:LED
- added D2: Yellow LED, LED_THT:LED_D1.8mm_W3.3mm_H2.4mm, symbol Device:LED
- added D3: Green LED, LED_THT:LED_D1.8mm_W3.3mm_H2.4mm, symbol Device:LED
- added J3: CXO TP, Connector_PinHeader_2.54mm:PinHeader_1x01_P2.54mm_Vertical, symbol Connector:Conn_01x01_Pin
- added R4, R5, R6: 330, Resistor_SMD:R_1206_3216Metric_Pad1.30x1.75mm_HandSolder, symbol Device:R_US
Connections:
- net GND: now also D1.1 (K), D2.1 (K), D3.1 (K)
- net at U13.10 (PC0): now also R4.1
- net at U13.11 (PC1): now also R5.1
- net at U13.12 (PC2): now also R6.1
- net at U4.22 (CLKOUT): now also J3.1 (Pin_1)
- new net: D2.2 (A), R5.2
- new net: D1.2 (A), R4.2
- new net: D3.2 (A), R6.2
- no-connect marks 41 -> 37
