File: can_tester/can_tester.kicad_sch (KiCad schematic)
At the start: 27 parts, among them J1 Conn_01x02_Pin, J10 USB to UART Conn, J3 CXO TP, J5 X9 LOCAL CAN Feedthrough Conn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, J6 X8: LOCAL CAN Host Interface, J7 Pins to select 120 terminal r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, J8 UPDI Friend Input Terminal, SW1 DIP Switch, U13 AVR128DB48x-xPT, U4 MCP25625 - CAN Transciever, Y2 Crystal_GND24

Commit message: so much! I should push more!
Parts:
- removed J5: X9 LOCAL CAN Feedthrough Connector, Connector_Dsub:DSUB-9_Pins_Horizontal_P2.77x2.84mm_EdgePinOffset9.40mm, symbol Connector:DE9_Pins
- added J13: CANL TP, Connector_PinHeader_2.54mm:PinHeader_1x02_P2.54mm_Vertical, symbol Connector:Conn_01x02_Pin
- added J14: CANH TP, Connector_PinHeader_2.54mm:PinHeader_1x02_P2.54mm_Vertical, symbol Connector:Conn_01x02_Pin
- added J15: FILT CANL TP, Connector_PinHeader_2.54mm:PinHeader_1x02_P2.54mm_Vertical, symbol Connector:Conn_01x02_Pin
- added J16: FILT CANH TP, Connector_PinHeader_2.54mm:PinHeader_1x02_P2.54mm_Vertical, symbol Connector:Conn_01x02_Pin
- added J17, J18: GND Conn, Connector_PinHeader_2.54mm:PinHeader_1x02_P2.54mm_Vertical, symbol Connector:Conn_01x02_Pin
- added J2: X9: LOCAL CAN Host Interface, dsub:CONN_DE09-SL-24_ADM_DSUB, symbol dsub_with_mounts:DE9_Pins
- C10, C9: footprint Capacitor_SMD:C_0603_1608Metric_Pad1.08x0.95mm_HandSolder -> Capacitor_SMD:C_1206_3216Metric_Pad1.33x1.80mm_HandSolder
- C13, C14, C15, C16, C17, C18: footprint Capacitor_SMD:C_0603_1608Metric_Pad1.08x0.95mm_HandSolder -> Capacitor_SMD:C_0805_2012Metric_Pad1.18x1.45mm_HandSolder
- J10: value USB to UART Conn -> USB to TTL Conn; footprint TerminalBlock:TerminalBlock_MaiXu_MX126-5.0-06P_1x06_P5.00mm -> Connector_PinHeader_2.54mm:PinHeader_1x06_P2.54mm_Vertical
- J6: footprint Connector_Dsub:DSUB-9_Pins_Horizontal_P2.77x2.84mm_EdgePinOffset9.40mm -> dsub:CONN_DE09-SL-24_ADM_DSUB
- J7: value Pins to select 120 terminal resistance or not -> Headers for terminal resistance; footprint TerminalBlock:TerminalBlock_MaiXu_MX126-5.0-03P_1x03_P5.00mm -> Connector_PinHeader_2.54mm:PinHeader_1x03_P2.54mm_Vertical
- R3: footprint Resistor_SMD:R_1206_3216Metric_Pad1.30x1.75mm_HandSolder -> Resistor_THT:R_Axial_DIN0204_L3.6mm_D1.6mm_P2.54mm_Vertical
Connections:
- net CAN H: now also J14.1 (Pin_1), J14.2 (Pin_2), J2.7
- net CAN H FILT: now also J16.1 (Pin_1), J16.2 (Pin_2)
- net CAN L: now also J13.1 (Pin_1), J13.2 (Pin_2), J2.2
- net CAN L FILT: now also J15.1 (Pin_1), J15.2 (Pin_2)
- net GND: now also J6.10, J6.11, U4.26 (V_{SS}), J17.1 (Pin_1), J17.2 (Pin_2), J18.1 (Pin_1), J18.2 (Pin_2), J2.10, J2.11, J2.3, J2.6; no longer U4.5 (STBY)
- net RESET: now also U13.46 (PA2)
- net at U13.22 (PD2): now also SW1.8; no longer SW1.4
- net at U13.23 (PD3): now also SW1.4; no longer SW1.1
- net at U13.24 (PD4): now also SW1.1; no longer SW1.8
- net Rx0: now reaches U13.6 (PB2)
- net Rx0: now also U4.12 (~{Rx0BF})
- net Rx1: now reaches U13.7 (PB3)
- net Rx1: now also U4.11 (~{Rx1BF})
- net STBY: now reaches U13.8 (PB4)
- net STBY: now also U4.5 (STBY)
- no-connect marks 37 -> 30
Other:
- note added: "Cable that allows for serial prints from AVR to PC over serial"
- note added: "Signifier LEDs. Can tie to whatever we see fit"
- note added: "Test point to check CXO frequency"
- note added: "These are perhaps ill advised 'hacky' ways of not having to make a doulbe sided board. PCB layout shows them as having a trace between them on the bottom, but this will be achieved by placing jumper across the header pins"
- note added: "This breakout board will be for writing code to AVR Middle pin should be 5V, but future proofing it for when we don't actually want that and AVR will get power elsewhere"
- note added: "Two header pins to provide easy test points for points we may want/need to debug. Easy for osc probes to be attached to."
- note removed: "This breakout board will be for writing code to AVR"
- moved on the sheet: D1, D2, D3, FL1, J10, J7, R3, R4, R5, R6
