File: adc_test_board/adc_test_board.kicad_sch (KiCad schematic)
At the start: 25 parts, among them J2 Conn_01x03_Pin, J3 Screw_Terminal_01x03, J4 PRT-14417, J6 Conn_01x03_Pin, J7 Conn_01x03_Pin, U1 LMC6082, U2 ADS1115IDGS, U3 REF3025, U4 5V LDO, U5 INA159AIDGKR

Commit message: so much! I should push more!
Parts:
- removed C1: 100p, Capacitor_THT:C_Disc_D3.0mm_W1.6mm_P2.50mm, symbol Device:C
- removed C3: 100n, Capacitor_SMD:C_1206_3216Metric, symbol Device:C
- removed C5: C_Polarized, Capacitor_SMD:CP_Elec_10x10.5, symbol Device:C_Polarized
- removed FB2: FerriteBead, Inductor_SMD:L_1206_3216Metric, symbol Device:FerriteBead
- removed J2: Conn_01x03_Pin, Connector_PinHeader_2.54mm:PinHeader_1x03_P2.54mm_Vertical, symbol Connector:Conn_01x03_Pin
- removed J3: Screw_Terminal_01x03, TerminalBlock_Phoenix:TerminalBlock_Phoenix_PTSM-0,5-3-2,5-V-SMD_1x03-1MP_P2.50mm_Vertical, symbol Connector:Screw_Terminal_01x03
- removed R1: 5G, Resistor_THT:R_Axial_DIN0204_L3.6mm_D1.6mm_P2.54mm_Vertical, symbol Device:R_US
- removed R10: 10k, Resistor_SMD:R_1206_3216Metric_Pad1.30x1.75mm_HandSolder, symbol Device:R_US
- removed R12, R2, R9: 1k, Resistor_SMD:R_1206_3216Metric_Pad1.30x1.75mm_HandSolder, symbol Device:R_US
- removed U1: LMC6082, Package_DIP:DIP-8_W7.62mm, symbol Amplifier_Operational:LMC6082
- added J1: Test voltage headers, Connector_PinHeader_2.54mm:PinHeader_1x02_P2.54mm_Vertical, symbol Connector:Conn_01x02_Pin
- added J2: Supply Input, Connector_PinHeader_2.54mm:PinHeader_1x02_P2.54mm_Vertical, symbol Connector:Conn_01x02_Pin
- added J8: Pins to decide which voltage is being checked., Connector_PinHeader_2.54mm:PinHeader_1x03_P2.54mm_Vertical, symbol Connector:Conn_01x03_Pin
Connections:
- net V_filt: now reaches C4.1, R11.2
- net V_filt: now also J8.1 (Pin_1)
- net Output renamed V_test
- net V_test: now also J8.2 (Pin_2)
- net V+ renamed V_in
- net V_in: now also J2.1 (Pin_1), J2.2 (Pin_2)
- new net V_unfilt: J1.1 (Pin_1), J1.2 (Pin_2), J8.3 (Pin_3)
Other:
- note added: "Filtering circuit present on the electrometer. Can only apply Positive voltage!!!!"
- note added: "For applying voltage from DC supply/FG or the like bypasses filtering circuit so we can look at negative voltage as well. double pins for easier alligator attachment. attach gnd clip to ground plane"
- note added: "Power rails from benchtop power supply Double header pin for easy alligator clip attachment attach ground to ground plane"
- note removed: "Electrometer - first stage is charge reading, second stage is for gain (unity or 10x based on header pins)"
- note removed: "Filtering circuit to give as clean of rails as possible to the Op Amp"
- note removed: "Power rails from benchtop power supply"
