File: electrometer_pcb/_restore_backup_2026-07-22T20-01-23-657/electrometer.kicad_sch (KiCad schematic)
At the start: 25 parts, among them J2 Conn_01x03_Pin, J3 Screw_Terminal_01x03, J4 PRT-14417, J6 Conn_01x03_Pin, J7 Conn_01x03_Pin, U1 LMC6082, U2 ADS1115IDGS, U3 REF3025, U4 5V LDO, U5 INA159AIDGKR

Commit message: so much! I should push more!
Parts:
- removed J6, J7: Conn_01x03_Pin, Connector_PinHeader_2.54mm:PinHeader_1x03_P2.54mm_Vertical, symbol Connector:Conn_01x03_Pin
- R11, R12: value 1k -> 10
Connections:
- net ADDR is gone; now on net GND: U2.1 (ADDR)
Other:
- note added: "Tying ADDR to GND makes the I2C address 1001000b"
- note removed: "Use jumpers to set I2C address GND 1001000b VDD 1001001b SDA (Blue) 1001010b SCL (Yellow) 1001011b"
