File: electrometer_for_spinning_disk_right_side/electrometer_for_spinning_disk_right_side.kicad_sch (KiCad schematic)
At the start: 21 parts, among them J2 Conn_01x03_Pin, J3 Screw_Terminal_01x03, J4 Screw_Terminal_01x03, U1 LMC6082, U3 REF3025, U5 INA159AIDGKR

Commit message: perfunctory commit
Parts:
- J3: footprint TerminalBlock_MetzConnect:TerminalBlock_MetzConnect_Type055_RT01503HDWU_1x03_P5.00mm_Horizontal -> TerminalBlock_Phoenix:TerminalBlock_Phoenix_PTSM-0,5-3-2,5-V-SMD_1x03-1MP_P2.50mm_Vertical
Changed lines of the file:
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@@
 		)
 		(instances
-			(project "electrometer_for_spinning_disk"
+			(project "electrometer_for_spinning_disk_right_side"
 				(path "/9f68a0c6-015a-4a20-8c62-b92ea580298b"
 					(reference "FB2")
@@
 		)
 		(instances
-			(project "electrometer_for_spinning_disk"
+			(project "electrometer_for_spinning_disk_right_side"
 				(path "/9f68a0c6-015a-4a20-8c62-b92ea580298b"
 					(reference "R12")
@@
 		)
 		(instances
-			(project "electrometer_for_spinning_disk"
+			(project "electrometer_for_spinning_disk_right_side"
 				(path "/9f68a0c6-015a-4a20-8c62-b92ea580298b"
 					(reference "#PWR022")
@@
 		)
 		(instances
-			(project "electrometer_for_spinning_disk"
+			(project "electrometer_for_spinning_disk_right_side"
 				(path "/9f68a0c6-015a-4a20-8c62-b92ea580298b"
 					(reference "#PWR015")
@@
 		)
 		(instances
-			(project "electrometer_for_spinning_disk"
+			(project "electrometer_for_spinning_disk_right_side"
 				(path "/9f68a0c6-015a-4a20-8c62-b92ea580298b"
 					(reference "#PWR016")
@@
 		)
 		(instances
-			(project "electrometer_for_spinning_disk"
+			(project "electrometer_for_spinning_disk_right_side"
 				(path "/9f68a0c6-015a-4a20-8c62-b92ea580298b"
 					(reference "R2")
@@
 		)
 		(instances
-			(project "electrometer_for_spinning_disk"
+			(project "electrometer_for_spinning_disk_right_side"
 				(path "/9f68a0c6-015a-4a20-8c62-b92ea580298b"
 					(reference "U5")
@@
 		)
 		(instances
-			(project "electrometer_for_spinning_disk"
+			(project "electrometer_for_spinning_disk_right_side"
 				(path "/9f68a0c6-015a-4a20-8c62-b92ea580298b"
 					(reference "U1")
@@
 		)
 		(instances
-			(project "electrometer_for_spinning_disk"
+			(project "electrometer_for_spinning_disk_right_side"
 				(path "/9f68a0c6-015a-4a20-8c62-b92ea580298b"
 					(reference "R9")
@@
 		)
 		(instances
-			(project "electrometer_for_spinning_disk"
+			(project "electrometer_for_spinning_disk_right_side"
 				(path "/9f68a0c6-015a-4a20-8c62-b92ea580298b"
 					(reference "C3")
@@
 		)
 		(instances
-			(project "electrometer_for_spinning_disk"
+			(project "electrometer_for_spinning_disk_right_side"
 				(path "/9f68a0c6-015a-4a20-8c62-b92ea580298b"
 					(reference "#PWR021")
@@
 		)
 		(instances
-			(project "electrometer_for_spinning_disk"
+			(project "electrometer_for_spinning_disk_right_side"
 				(path "/9f68a0c6-015a-4a20-8c62-b92ea580298b"
 					(reference "#PWR018")
@@
 		)
 		(instances
-			(project "electrometer_for_spinning_disk"
+			(project "electrometer_for_spinning_disk_right_side"
 				(path "/9f68a0c6-015a-4a20-8c62-b92ea580298b"
 					(reference "#PWR017")
@@
 		)
 		(instances
-			(project "electrometer_for_spinning_disk"
+			(project "electrometer_for_spinning_disk_right_side"
 				(path "/9f68a0c6-015a-4a20-8c62-b92ea580298b"
 					(reference "U1")
@@
 		)
 		(instances
-			(project "electrometer_for_spinning_disk"
+			(project "electrometer_for_spinning_disk_right_side"
 				(path "/9f68a0c6-015a-4a20-8c62-b92ea580298b"
 					(reference "#PWR08")
@@
 		)
 		(instances
-			(project "electrometer_for_spinning_disk"
+			(project "electrometer_for_spinning_disk_right_side"
 				(path "/9f68a0c6-015a-4a20-8c62-b92ea580298b"
 					(reference "J4")
@@
 		)
 		(instances
-			(project "electrometer_for_spinning_disk"
+			(project "electrometer_for_spinning_disk_right_side"
 				(path "/9f68a0c6-015a-4a20-8c62-b92ea580298b"
 					(reference "#PWR06")
@@
 		)
 		(instances
-			(project "electrometer_for_spinning_disk"
+			(project "electrometer_for_spinning_disk_right_side"
 				(path "/9f68a0c6-015a-4a20-8c62-b92ea580298b"
 					(reference "#PWR012")
@@
 		)
 		(instances
-			(project "electrometer_for_spinning_disk"
+			(project "electrometer_for_spinning_disk_right_side"
 				(path "/9f68a0c6-015a-4a20-8c62-b92ea580298b"
 					(reference "FB1")
@@
 		)
 		(instances
-			(project "electrometer_for_spinning_disk"
+			(project "electrometer_for_spinning_disk_right_side"
 				(path "/9f68a0c6-015a-4a20-8c62-b92ea580298b"
 					(reference "C4")
@@
 		)
 		(instances
-			(project "electrometer_for_spinning_disk"
+			(project "electrometer_for_spinning_disk_right_side"
 				(path "/9f68a0c6-015a-4a20-8c62-b92ea580298b"
 					(reference "J2")
@@
 		)
 		(instances
-			(project "electrometer_for_spinning_disk"
+			(project "electrometer_for_spinning_disk_right_side"
 				(path "/9f68a0c6-015a-4a20-8c62-b92ea580298b"
 					(reference "R11")
@@
 		)
 		(instances
-			(project "electrometer_for_spinning_disk"
+			(project "electrometer_for_spinning_disk_right_side"
 				(path "/9f68a0c6-015a-4a20-8c62-b92ea580298b"
 					(reference "#PWR02")
@@
 		)
 		(instances
-			(project "electrometer_for_spinning_disk"
+			(project "electrometer_for_spinning_disk_right_side"
 				(path "/9f68a0c6-015a-4a20-8c62-b92ea580298b"
 					(reference "#PWR09")
@@
 		)
 		(instances
-			(project "electrometer_for_spinning_disk"
+			(project "electrometer_for_spinning_disk_right_side"
 				(path "/9f68a0c6-015a-4a20-8c62-b92ea580298b"
 					(reference "#PWR05")
@@
 		)
 		(instances
-			(project "electrometer_for_spinning_disk"
+			(project "electrometer_for_spinning_disk_right_side"
 				(path "/9f68a0c6-015a-4a20-8c62-b92ea580298b"
 					(reference "R10")
@@
 		)
 		(instances
-			(project "electrometer_for_spinning_disk"
+			(project "electrometer_for_spinning_disk_right_side"
 				(path "/9f68a0c6-015a-4a20-8c62-b92ea580298b"
 					(reference "#PWR019")
@@
 		)
 		(instances
-			(project "electrometer_for_spinning_disk"
+			(project "electrometer_for_spinning_disk_right_side"
 				(path "/9f68a0c6-015a-4a20-8c62-b92ea580298b"
 					(reference "U3")
@@
 		)
 		(instances
-			(project "electrometer_for_spinning_disk"
+			(project "electrometer_for_spinning_disk_right_side"
 				(path "/9f68a0c6-015a-4a20-8c62-b92ea580298b"
 					(reference "#PWR014")
@@
 		)
 		(instances
-			(project "electrometer_for_spinning_disk"
+			(project "electrometer_for_spinning_disk_right_side"
 				(path "/9f68a0c6-015a-4a20-8c62-b92ea580298b"
 					(reference "C1")
@@
 		)
 		(instances
-			(project "electrometer_for_spinning_disk"
+			(project "electrometer_for_spinning_disk_right_side"
 				(path "/9f68a0c6-015a-4a20-8c62-b92ea580298b"
 					(reference "#PWR07")
@@
 		)
 		(instances
-			(project "electrometer_for_spinning_disk"
+			(project "electrometer_for_spinning_disk_right_side"
 				(path "/9f68a0c6-015a-4a20-8c62-b92ea580298b"
 					(reference "U1")
@@
 		)
 		(instances
-			(project "electrometer_for_spinning_disk"
+			(project "electrometer_for_spinning_disk_right_side"
 				(path "/9f68a0c6-015a-4a20-8c62-b92ea580298b"
 					(reference "C7")
@@
 		)
 		(instances
-			(project "electrometer_for_spinning_disk"
+			(project "electrometer_for_spinning_disk_right_side"
 				(path "/9f68a0c6-015a-4a20-8c62-b92ea580298b"
 					(reference "#PWR020")
@@
 		)
 		(instances
-			(project "electrometer_for_spinning_disk"
+			(project "electrometer_for_spinning_disk_right_side"
 				(path "/9f68a0c6-015a-4a20-8c62-b92ea580298b"
 					(reference "#PWR010")
@@
 		)
 		(instances
-			(project "electrometer_for_spinning_disk"
+			(project "electrometer_for_spinning_disk_right_side"
 				(path "/9f68a0c6-015a-4a20-8c62-b92ea580298b"
 					(reference "C6")
@@
 		)
 		(instances
-			(project "electrometer_for_spinning_disk"
+			(project "electrometer_for_spinning_disk_right_side"
 				(path "/9f68a0c6-015a-4a20-8c62-b92ea580298b"
 					(reference "R1")
@@
 		)
 		(instances
-			(project "electrometer_for_spinning_disk"
+			(project "electrometer_for_spinning_disk_right_side"
 				(path "/9f68a0c6-015a-4a20-8c62-b92ea580298b"
 					(reference "C2")
@@
 		)
 		(instances
-			(project "electrometer_for_spinning_disk"
+			(project "electrometer_for_spinning_disk_right_side"
 				(path "/9f68a0c6-015a-4a20-8c62-b92ea580298b"
 					(reference "C5")
@@
 		)
 		(instances
-			(project "electrometer_for_spinning_disk"
+			(project "electrometer_for_spinning_disk_right_side"
 				(path "/9f68a0c6-015a-4a20-8c62-b92ea580298b"
 					(reference "#PWR011")
@@
 			)
 		)
-		(property "Footprint" "TerminalBlock_MetzConnect:TerminalBlock_MetzConnect_Type055_RT01503HDWU_1x03_P5.00mm_Horizontal"
+		(property "Footprint" "TerminalBlock_Phoenix:TerminalBlock_Phoenix_PTSM-0,5-3-2,5-V-SMD_1x03-1MP_P2.50mm_Vertical"
 			(at 50.8 91.44 0)
 			(hide yes)
@@
 		)
 		(instances
-			(project "electrometer_for_spinning_disk"
+			(project "electrometer_for_spinning_disk_right_side"
 				(path "/9f68a0c6-015a-4a20-8c62-b92ea580298b"
 					(reference "J3")
@@
 		)
 		(instances
-			(project "electrometer_for_spinning_disk"
+			(project "electrometer_for_spinning_disk_right_side"
 				(path "/9f68a0c6-015a-4a20-8c62-b92ea580298b"
 					(reference "#PWR04")
@@
 		)
 		(instances
-			(project "electrometer_for_spinning_disk"
+			(project "electrometer_for_spinning_disk_right_side"
 				(path "/9f68a0c6-015a-4a20-8c62-b92ea580298b"
 					(reference "#PWR03")
