File: electrometer_pcb/electrometer.kicad_pcb (KiCad board)
At the start: 2 copper layers, 64.9 x 82 mm, 27 parts, among them J2 Conn_01x03_Pin, J3 Screw_Terminal_01x03, J4 PRT-14417, U1 LMC6082, U2 ADS1115IDGS, U3 REF3025, U4 5V LDO, U5 INA159AIDGKR

Commit message: so much! I should push more!
Parts:
- added J6: Conn_01x03_Pin, Connector_PinHeader_2.54mm:PinHeader_1x03_P2.54mm_Vertical, F.Cu at (130.6, 44.3)
- added J7: Conn_01x03_Pin, Connector_PinHeader_2.54mm:PinHeader_1x03_P2.54mm_Vertical, F.Cu at (128.1, 46.9)
- moved U2 0.18 mm to (120.0, 65.2)
Connections:
- U2 pad 1: GND -> /ADDR
Routing:
- net GND: track 217.2 -> 264.5 mm
- net /ADDR: track 0.00 -> 36.4 mm
- net /Yellow: track 3.91 -> 29.4 mm
- net /Blue: track 3.71 -> 19.8 mm
- net +3.3V: track 3.90 -> 19.8 mm
- net Net-(J2-Pin_2): track 23.3 -> 26.4 mm
Other:
- board text added: "GND"
- board text added: "SCL"
- board text added: "SDA"
- board text added: "VDD"

Commit message: lots of new stuff
Parts:
- moved J6 15.0 mm to (135.5, 58.5)
- moved J7 15.0 mm to (132.9, 61.0)
- moved REF** 11.6 mm to (104.0, 53.0)
- moved REF** 11.6 mm to (104.0, 107.0)
- moved REF** 9.89 mm to (137.0, 53.0)
- moved REF** 9.89 mm to (137.0, 107.0)
Routing:
- net GND: track 264.5 -> 253.0 mm
- net /ADDR: track 36.4 -> 25.6 mm
- net /Yellow: track 29.4 -> 22.9 mm
- net +3.3V: track 19.8 -> 21.8 mm
Other:
- board size 64.9 x 82 mm -> 43 x 60 mm
- board text removed: "GND"
- board text removed: "SCL"
- board text removed: "SDA"
- board text removed: "VDD"
Changed lines of the file:
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@@
 	(footprint "Connector_PinHeader_2.54mm:PinHeader_1x03_P2.54mm_Vertical"
 		(layer "F.Cu")
-		(at 128.06 46.86 90)
+		(at 132.92 61 90)
 		(descr "Through hole straight pin header, 1x03, 2.54mm pitch, single row")
 		(tags "Through hole pin header THT 1x03 2.54mm single row")
@@
 	(footprint "Connector_PinHeader_2.54mm:PinHeader_1x03_P2.54mm_Vertical"
 		(layer "F.Cu")
-		(at 130.6 44.32)
+		(at 135.46 58.46)
 		(descr "Through hole straight pin header, 1x03, 2.54mm pitch, single row")
 		(tags "Through hole pin header THT 1x03 2.54mm single row")
@@
 		(pad "2" thru_hole circle
 			(at 2.54 0 90)
-			(size 2 2)
-			(drill 0.7)
+			(size 2.2 2.2)
+			(drill 1.2)
 			(layers "*.Cu" "*.Mask")
 			(remove_unused_layers no)
@@
 	(footprint "MountingHole:MountingHole_2.7mm"
 		(layer "F.Cu")
-		(at 94.450001 113.499999)
+		(at 104 107)
 		(descr "Mounting Hole 2.7mm, no annular")
 		(tags "mounting hole 2.7mm no annular")
@@
 	(footprint "MountingHole:MountingHole_2.7mm"
 		(layer "F.Cu")
-		(at 144.450001 46.499999)
+		(at 137 53)
 		(descr "Mounting Hole 2.7mm, no annular")
 		(tags "mounting hole 2.7mm no annular")
@@
 	(footprint "MountingHole:MountingHole_2.7mm"
 		(layer "F.Cu")
-		(at 94.450001 46.499999)
+		(at 104 53)
 		(descr "Mounting Hole 2.7mm, no annular")
 		(tags "mounting hole 2.7mm no annular")
@@
 	(footprint "MountingHole:MountingHole_2.7mm"
 		(layer "F.Cu")
-		(at 144.450001 113.499999)
+		(at 137 107)
 		(descr "Mounting Hole 2.7mm, no annular")
 		(tags "mounting hole 2.7mm no annular")
@@
 	)
 	(gr_rect
-		(start 87.05 38.999998)
-		(end 151.950001 120.999998)
+		(start 99 50)
+		(end 141.999999 110)
 		(stroke
 			(width 0.1)
@@
 		(layer "Edge.Cuts")
 	)
-	(gr_text "SDA"
-		(at 120.46 47.86 0)
-		(layer "F.Cu")
-		(effects
-			(font
-				(size 2 2)
-				(thickness 0.5)
-				(bold yes)
-			)
-			(justify left bottom)
-		)
-	)
-	(gr_text "SCL"
-		(at 127.66 42.26 0)
-		(layer "F.Cu")
-		(effects
-			(font
-				(size 2 2)
-				(thickness 0.5)
-				(bold yes)
-			)
-			(justify left bottom)
-		)
-	)
-	(gr_text "VDD\n"
-		(at 127.8 53.8 0)
-		(layer "F.Cu")
-		(effects
-			(font
-				(size 2 2)
-				(thickness 0.5)
-				(bold yes)
-			)
-			(justify left bottom)
-		)
-	)
-	(gr_text "GND"
-		(at 134.86 48.06 0)
+	(gr_text "10x"
+		(at 133 86 0)
 		(layer "F.Cu")
 		(effects
@@
 	)
 	(gr_text "1x"
-		(at 138.014461 74.929999 0)
-		(layer "F.Cu")
-		(effects
-			(font
-				(size 2 2)
-				(thickness 0.5)
-				(bold yes)
-			)
-			(justify left bottom)
-		)
-	)
-	(gr_text "10x"
-		(at 138.014461 80.729999 0)
+		(at 134 71 0)
 		(layer "F.Cu")
 		(effects
@@
 	)
 	(segment
+		(start 132.427107 70.279999)
+		(end 129.389461 70.279999)
+		(width 0.3)
+		(layer "F.Cu")
+		(net "GND")
+	)
+	(segment
 		(start 103.064461 98.379999)
 		(end 106.014461 101.329999)
@@
 	)
 	(segment
-		(start 134.571822 48.291822)
-		(end 134.571822 65.097638)
-		(width 0.3)
-		(layer "F.Cu")
-		(net "GND")
-	)
-	(segment
 		(start 108.726961 104.042499)
 		(end 118.701961 104.042499)
@@
 	)
 	(segment
-		(start 133.14 46.86)
-		(end 134.571822 48.291822)
-		(width 0.3)
-		(layer "F.Cu")
-		(net "GND")
-	)
-	(segment
 		(start 126.929999 59.529999)
 		(end 121.450001 59.529999)
@@
 	)
 	(segment
+		(start 138 64.707106)
+		(end 132.427107 70.279999)
+		(width 0.3)
+		(layer "F.Cu")
+		(net "GND")
+	)
+	(segment
 		(start 130.901961 104.042499)
 		(end 133.614461 101.329999)
@@
 	)
 	(segment
+		(start 138 61)
+		(end 138 64.707106)
+		(width 0.3)
+		(layer "F.Cu")
+		(net "GND")
+	)
+	(segment
 		(start 121.22383 64.175)
 		(end 112.175 64.175)
@@
 	)
 	(segment
-		(start 134.571822 65.097638)
-		(end 129.389461 70.279999)
-		(width 0.3)
-		(layer "F.Cu")
-		(net "GND")
-	)
-	(segment
 		(start 128.139461 65.260539)
 		(end 128.370001 65.029999)
@@
 	)
 	(segment
-		(start 119.462501 59.542499)
-		(end 119.450001 59.529999)
+		(start 120.300002 57.904999)
+		(end 129.824999 57.904999)
 		(width 0.3)
 		(layer "F.Cu")
@@
 	)
 	(segment
-		(start 119.450001 59.529999)
-		(end 119.450001 56.349999)
+		(start 119.462501 59.542499)
+		(end 119.450001 59.529999)
 		(width 0.3)
 		(layer "F.Cu")
@@
 	)
 	(segment
-		(start 128.06 47.74)
-		(end 128.06 46.86)
+		(start 119.450001 59.529999)
+		(end 119.450001 58.755)
 		(width 0.3)
 		(layer "F.Cu")
@@
 	)
 	(segment
-		(start 119.450001 56.349999)
-		(end 128.06 47.74)
+		(start 119.450001 58.755)
+		(end 120.300002 57.904999)
 		(width 0.3)
 		(layer "F.Cu")
@@
 	)
 	(segment
-		(start 134.071822 62.779745)
-		(end 134.071822 50.331822)
+		(start 129.824999 57.904999)
+		(end 132.92 61)
 		(width 0.3)
 		(layer "F.Cu")
-		(net "/ADDR")
+		(net "/Blue")
 	)
 	(segment
-		(start 127.539461 69.202181)
-		(end 128.241642 68.5)
+		(start 135.46 61)
+		(end 137 62.54)
 		(width 0.3)
 		(layer "F.Cu")
@@
 	)
 	(segment
-		(start 128.241642 68.5)
-		(end 128.351567 68.5)
+		(start 137 62.54)
+		(end 137 65)
 		(width 0.3)
 		(layer "F.Cu")
@@
 	)
 	(segment
-		(start 128.351567 68.5)
-		(end 134.071822 62.779745)
+		(start 133.35 68.65)
+		(end 122.457106 68.65)
 		(width 0.3)
 		(layer "F.Cu")
@@
 	(segment
 		(start 118.95 68.17812)
-		(end 119.974061 69.202181)
+		(end 118.95 67.35)
 		(width 0.3)
 		(layer "F.Cu")
@@
 	)
 	(segment
-		(start 119.974061 69.202181)
-		(end 127.539461 69.202181)
+		(start 122.002107 69.104999)
+		(end 119.876879 69.104999)
 		(width 0.3)
 		(layer "F.Cu")
@@
 	)
 	(segment
-		(start 134.071822 50.331822)
-		(end 130.6 46.86)
+		(start 137 65)
+		(end 133.35 68.65)
 		(width 0.3)
 		(layer "F.Cu")
@@
 	)
 	(segment
-		(start 118.95 67.35)
+		(start 122.457106 68.65)
+		(end 122.002107 69.104999)
+		(width 0.3)
+		(layer "F.Cu")
+		(net "/ADDR")
+	)
+	(segment
+		(start 119.876879 69.104999)
 		(end 118.95 68.17812)
 		(width 0.3)
@@
 	)
 	(segment
-		(start 118.450001 47.149999)
-		(end 121.28 44.32)
+		(start 118.95 63.05)
+		(end 118.450001 62.550001)
 		(width 0.3)
 		(layer "F.Cu")
@@
 	)
 	(segment
-		(start 121.28 44.32)
-		(end 130.6 44.32)
+		(start 118.450001 59.529999)
+		(end 118.450001 58.099543)
 		(width 0.3)
 		(layer "F.Cu")
@@
 	)
 	(segment
-		(start 118.95 63.05)
-		(end 118.450001 62.550001)
+		(start 118.450001 58.099543)
+		(end 119.144545 57.404999)
 		(width 0.3)
 		(layer "F.Cu")
@@
 	)
 	(segment
-		(start 118.450001 59.529999)
-		(end 118.450001 47.149999)
+		(start 119.144545 57.404999)
+		(end 134.404999 57.404999)
 		(width 0.3)
 		(layer "F.Cu")
@@
 	)
 	(segment
-		(start 120.450001 60.016261)
-		(end 120.450001 59.529999)
+		(start 134.404999 57.404999)
+		(end 135.46 58.46)
 		(width 0.3)
 		(layer "F.Cu")
-		(net "+3.3V")
+		(net "/Yellow")
 	)
 	(segment
-		(start 120.450001 58.599543)
-		(end 121.649544 57.4)
+		(start 120.450001 60.016261)
+		(end 120.450001 59.529999)
 		(width 0.3)
 		(layer "F.Cu")
@@
 	)
 	(segment
-		(start 120.450001 59.529999)
-		(end 120.450001 58.599543)
+		(start 127.924999 58.404999)
+		(end 120.800002 58.404999)
 		(width 0.3)
 		(layer "F.Cu")
@@
 	)
 	(segment
-		(start 121.649544 57.4)
-		(end 123.4 57.4)
+		(start 133.06 63.54)
+		(end 127.924999 58.404999)
 		(width 0.3)
 		(layer "F.Cu")
@@
 	)
 	(segment
-		(start 123.4 57.4)
-		(end 127.628325 53.171675)
+		(start 135.46 63.54)
+		(end 133.06 63.54)
 		(width 0.3)
 		(layer "F.Cu")
@@
 	)
 	(segment
-		(start 129.437919 49.4)
-		(end 130.6 49.4)
-		(width 0.3)
-		(layer "F.Cu")
-		(net "+3.3V")
-	)
-	(segment
-		(start 127.628325 51.209594)
-		(end 129.437919 49.4)
+		(start 120.450001 58.755)
+		(end 120.450001 59.529999)
 		(width 0.3)
 		(layer "F.Cu")
@@
 	)
 	(segment
-		(start 127.628325 53.171675)
-		(end 127.628325 51.209594)
+		(start 120.800002 58.404999)
+		(end 120.450001 58.755)
 		(width 0.3)
 		(layer "F.Cu")
