File: power_board_disk/power_board_disk.kicad_pcb (KiCad board)
At the start: 2 copper layers, 119 x 32 mm, 30 parts, among them J1 Oscillation Setting, J2 Electro Power1, J3 Capacitance Osc, J5 Inductive Charging, J6 Screw_Terminal_01x04, J7 Electro Power2, U1 TC7660 - Charge Pump, U2 ADS1115IDGS, U3 XIAO ESP32C3

Commit message: lots of new stuff
Parts:
- added J4: -5V Test Point, Connector_PinHeader_2.54mm:PinHeader_1x02_P2.54mm_Vertical, F.Cu at (94.3, 97.2)
- C1, C2: value 4.7uF -> 10uF; footprint Capacitor_Tantalum_SMD:CP_EIA-3216-18_Kemet-A_HandSolder -> Capacitor_THT:CP_Radial_D4.0mm_P2.00mm
- moved C5 37.6 mm to (135.6, 73.2)
- moved C6 37.6 mm to (114.4, 93.3)
- moved C7 37.6 mm to (111.7, 93.3)
- moved C8 37.6 mm to (108.9, 93.3)
- moved D2 37.6 mm to (181.3, 76.5)
- moved D3 37.6 mm to (181.3, 81.3)
- moved D4 37.6 mm to (181.1, 86.1)
- moved J1 37.6 mm to (114.3, 86.4)
- moved J2 37.6 mm to (188.5, 91.5)
- moved J3 37.6 mm to (114.3, 88.9)
- moved J5 37.6 mm to (112.7, 75.9)
- moved J6 37.6 mm to (151.0, 97.5)
- moved J7 37.6 mm to (77.5, 91.5)
- moved R4 37.6 mm to (173.0, 77.0)
- moved R5 37.6 mm to (173.0, 81.3)
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Routing:
- net -5V: track 142.0 -> 152.7 mm
- net GND: track 161.0 -> 163.5 mm
- net Net-(U1-CAP+): track 3.17 -> 5.30 mm
- net Net-(U1-CAP-): track 3.22 -> 5.27 mm
